File: util-BleedAFuzz.kicad_pcb (KiCad board)
At the start: 2 copper layers, 9.5 x 21.2 mm, 5 parts, among them J1 Conn_01x03_Pin, Q1 BC847

Commit message: util-BleedAFuzz 0.2 fab outputs (g2)
Parts:
- RV1: moved to B.Cu
- moved R1 7.44 mm to (97.7, 84.2), turned to 90 degrees
- moved R2 7.14 mm to (103.4, 84.2), turned to 90 degrees
- moved RV1 6.00 mm to (100.5, 80.0), turned to 180 degrees
- moved Q1 0.10 mm to (100.4, 83.3), turned to 90 degrees
Routing:
- net EMITTER: track 0.00 -> 8.40 mm
- net Net-(R2-Pad2): track 7.86 -> 0.00 mm
- net COLLECTOR: track 9.32 -> 17.1 mm
- net BASE: track 6.04 -> 9.43 mm
- removed copper zone on B.Cu, net BASE
- removed copper zone on F.Cu, net EMITTER
- removed copper zone on B.Cu, net Net-(R2-Pad2)
Other:
- board size 9.5 x 21.2 mm -> 9.5 x 14.7 mm
